Commit message: Rename wheeled robot project name

File: src/wheeled_robot/urdf/kuka_lwr.urdf.xacro (robot description, xacro)
@@ -6,5 +6,5 @@
     <visual>
       <geometry>
-        <mesh filename="package://wheeled_robot_urdf/meshes/arm_base.dae" scale="${1/size_factor} ${1/size_factor} ${1/size_factor}" />
+        <mesh filename="package://wheeled_robot/meshes/arm_base.dae" scale="${1/size_factor} ${1/size_factor} ${1/size_factor}" />
       </geometry>
       <material name="Orange" />
@@ -23,5 +23,5 @@
       <origin rpy="0 0 ${pi}" />
       <geometry>
-        <mesh filename="package://wheeled_robot_urdf/meshes/arm_segment_a.dae" scale="${1/size_factor} ${1/size_factor} ${1/size_factor}" />
+        <mesh filename="package://wheeled_robot/meshes/arm_segment_a.dae" scale="${1/size_factor} ${1/size_factor} ${1/size_factor}" />
       </geometry>
       <material name="Orange" />
@@ -29,5 +29,5 @@
     <collision>
       <geometry>
-        <mesh filename="package://wheeled_robot_urdf/meshes/arm_segment_a.dae" scale="${1/size_factor} ${1/size_factor} ${1/size_factor}" />
+        <mesh filename="package://wheeled_robot/meshes/arm_segment_a.dae" scale="${1/size_factor} ${1/size_factor} ${1/size_factor}" />
       </geometry>
     </collision>
@@ -44,5 +44,5 @@
       <origin xyz="0 0 ${0.2/size_factor}" rpy="${pi} 0 ${pi}" />
       <geometry>
-        <mesh filename="package://wheeled_robot_urdf/meshes/arm_segment_b.dae" scale="${1/size_factor} ${1/size_factor} ${1/size_factor}" />
+        <mesh filename="package://wheeled_robot/meshes/arm_segment_b.dae" scale="${1/size_factor} ${1/size_factor} ${1/size_factor}" />
       </geometry>
       <material name="Orange" />
@@ -51,5 +51,5 @@
       <origin xyz="0 0 ${0.2/size_factor}" rpy="${pi} 0 ${pi}" />
       <geometry>
-        <mesh filename="package://wheeled_robot_urdf/meshes/arm_segment_b.dae" scale="${1/size_factor} ${1/size_factor} ${1/size_factor}" />
+        <mesh filename="package://wheeled_robot/meshes/arm_segment_b.dae" scale="${1/size_factor} ${1/size_factor} ${1/size_factor}" />
       </geometry>
     </collision>
@@ -65,5 +65,5 @@
     <visual>
       <geometry>
-        <mesh filename="package://wheeled_robot_urdf/meshes/arm_segment_a.dae" scale="${1/size_factor} ${1/size_factor} ${1/size_factor}" />
+        <mesh filename="package://wheeled_robot/meshes/arm_segment_a.dae" scale="${1/size_factor} ${1/size_factor} ${1/size_factor}" />
       </geometry>
       <material name="Orange" />
@@ -71,5 +71,5 @@
     <collision>
       <geometry>
-        <mesh filename="package://wheeled_robot_urdf/meshes/arm_segment_a.dae" scale="${1/size_factor} ${1/size_factor} ${1/size_factor}" />
+        <mesh filename="package://wheeled_robot/meshes/arm_segment_a.dae" scale="${1/size_factor} ${1/size_factor} ${1/size_factor}" />
       </geometry>
     </collision>
@@ -86,5 +86,5 @@
       <origin xyz="0 0 ${0.2/size_factor}" rpy="0 ${pi} ${pi}" />
       <geometry>
-        <mesh filename="package://wheeled_robot_urdf/meshes/arm_segment_b.dae" scale="${1/size_factor} ${1/size_factor} ${1/size_factor}" />
+        <mesh filename="package://wheeled_robot/meshes/arm_segment_b.dae" scale="${1/size_factor} ${1/size_factor} ${1/size_factor}" />
       </geometry>
       <material name="Orange" />
@@ -92,5 +92,5 @@
     <collision>
       <geometry>
-        <mesh filename="package://wheeled_robot_urdf/meshes/arm_segment_b.dae" scale="${1/size_factor} ${1/size_factor} ${1/size_factor}" />
+        <mesh filename="package://wheeled_robot/meshes/arm_segment_b.dae" scale="${1/size_factor} ${1/size_factor} ${1/size_factor}" />
       </geometry>
     </collision>
@@ -107,5 +107,5 @@
       <origin rpy="0 0 ${pi}" />
       <geometry>
-        <mesh filename="package://wheeled_robot_urdf/meshes/arm_segment_last.dae" scale="${1/size_factor} ${1/size_factor} ${1/size_factor}" />
+        <mesh filename="package://wheeled_robot/meshes/arm_segment_last.dae" scale="${1/size_factor} ${1/size_factor} ${1/size_factor}" />
       </geometry>
       <material name="Orange"/>
@@ -113,5 +113,5 @@
     <collision>
       <geometry>
-        <mesh filename="package://wheeled_robot_urdf/meshes/arm_segment_last.dae" scale="${1/size_factor} ${1/size_factor} ${1/size_factor}" />
+        <mesh filename="package://wheeled_robot/meshes/arm_segment_last.dae" scale="${1/size_factor} ${1/size_factor} ${1/size_factor}" />
       </geometry>
     </collision>
@@ -128,5 +128,5 @@
       <origin rpy="0 0 ${pi}" />
       <geometry>
-        <mesh filename="package://wheeled_robot_urdf/meshes/arm_wrist.dae" scale="${1/size_factor} ${1/size_factor} ${1/size_factor}" />
+        <mesh filename="package://wheeled_robot/meshes/arm_wrist.dae" scale="${1/size_factor} ${1/size_factor} ${1/size_factor}" />
       </geometry>
       <material name="Grey"/>
@@ -134,5 +134,5 @@
     <collision>
       <geometry>
-        <mesh filename="package://wheeled_robot_urdf/meshes/arm_wrist.dae" scale="${1/size_factor} ${1/size_factor} ${1/size_factor}" />
+        <mesh filename="package://wheeled_robot/meshes/arm_wrist.dae" scale="${1/size_factor} ${1/size_factor} ${1/size_factor}" />
       </geometry>
     </collision>
@@ -149,5 +149,5 @@
       <origin rpy="0 0 ${pi}" />
       <geometry>
-        <mesh filename="package://wheeled_robot_urdf/meshes/arm_flanche.dae" scale="${1/size_factor} ${1/size_factor} ${1/size_factor}" />
+        <mesh filename="package://wheeled_robot/meshes/arm_flanche.dae" scale="${1/size_factor} ${1/size_factor} ${1/size_factor}" />
       </geometry>
       <material name="Grey"/>
@@ -155,5 +155,5 @@
     <collision>
       <geometry>
-        <mesh filename="package://wheeled_robot_urdf/meshes/arm_flanche.dae" scale="${1/size_factor} ${1/size_factor} ${1/size_factor}" />
+        <mesh filename="package://wheeled_robot/meshes/arm_flanche.dae" scale="${1/size_factor} ${1/size_factor} ${1/size_factor}" />
       </geometry>
     </collision>

File: src/wheeled_robot/urdf/wheeled_robot.urdf.xacro (robot description, xacro)
@@ -9,5 +9,5 @@
   <xacro:property name="body_height" value="0.3" />
   <xacro:property name="use_mesh_body" value="True" />
-  <xacro:property name="mesh_filename" value="package://wheeled_robot_urdf/meshes/chassis.dae" />
+  <xacro:property name="mesh_filename" value="package://wheeled_robot/meshes/chassis.dae" />
   <xacro:property name="side_wheel_mass" value="1" />
   <xacro:property name="side_wheel_length" value="0.04" />
@@ -117,5 +117,5 @@
   </joint>
   <!-- KUKA LWR -->
-  <xacro:include filename="$(find wheeled_robot_urdf)/urdf/kuka_lwr.urdf.xacro" />
+  <xacro:include filename="$(find wheeled_robot)/urdf/kuka_lwr.urdf.xacro" />
   <joint name="base_to_manipulator" type="fixed">
     <parent link="base_link" />
