Commit message: Finish tasks 1 and 2

File: src/wheeled_robot/wheelbot_description/urdf/kuka_lwr.xacro (robot description, xacro)
@@ -6,5 +6,5 @@
     <visual>
       <geometry>
-        <mesh filename="package://wheeled_robot/meshes/arm_base.dae" scale="${1/size_factor} ${1/size_factor} ${1/size_factor}" />
+        <mesh filename="package://wheelbot_description/meshes/arm_base.dae" scale="${1/size_factor} ${1/size_factor} ${1/size_factor}" />
       </geometry>
       <material name="Orange" />
@@ -23,5 +23,5 @@
       <origin rpy="0 0 ${pi}" />
       <geometry>
-        <mesh filename="package://wheeled_robot/meshes/arm_segment_a.dae" scale="${1/size_factor} ${1/size_factor} ${1/size_factor}" />
+        <mesh filename="package://wheelbot_description/meshes/arm_segment_a.dae" scale="${1/size_factor} ${1/size_factor} ${1/size_factor}" />
       </geometry>
       <material name="Orange" />
@@ -29,5 +29,5 @@
     <collision>
       <geometry>
-        <mesh filename="package://wheeled_robot/meshes/arm_segment_a.dae" scale="${1/size_factor} ${1/size_factor} ${1/size_factor}" />
+        <mesh filename="package://wheelbot_description/meshes/arm_segment_a.dae" scale="${1/size_factor} ${1/size_factor} ${1/size_factor}" />
       </geometry>
     </collision>
@@ -44,5 +44,5 @@
       <origin xyz="0 0 ${0.2/size_factor}" rpy="${pi} 0 ${pi}" />
       <geometry>
-        <mesh filename="package://wheeled_robot/meshes/arm_segment_b.dae" scale="${1/size_factor} ${1/size_factor} ${1/size_factor}" />
+        <mesh filename="package://wheelbot_description/meshes/arm_segment_b.dae" scale="${1/size_factor} ${1/size_factor} ${1/size_factor}" />
       </geometry>
       <material name="Orange" />
@@ -51,5 +51,5 @@
       <origin xyz="0 0 ${0.2/size_factor}" rpy="${pi} 0 ${pi}" />
       <geometry>
-        <mesh filename="package://wheeled_robot/meshes/arm_segment_b.dae" scale="${1/size_factor} ${1/size_factor} ${1/size_factor}" />
+        <mesh filename="package://wheelbot_description/meshes/arm_segment_b.dae" scale="${1/size_factor} ${1/size_factor} ${1/size_factor}" />
       </geometry>
     </collision>
@@ -65,5 +65,5 @@
     <visual>
       <geometry>
-        <mesh filename="package://wheeled_robot/meshes/arm_segment_a.dae" scale="${1/size_factor} ${1/size_factor} ${1/size_factor}" />
+        <mesh filename="package://wheelbot_description/meshes/arm_segment_a.dae" scale="${1/size_factor} ${1/size_factor} ${1/size_factor}" />
       </geometry>
       <material name="Orange" />
@@ -71,5 +71,5 @@
     <collision>
       <geometry>
-        <mesh filename="package://wheeled_robot/meshes/arm_segment_a.dae" scale="${1/size_factor} ${1/size_factor} ${1/size_factor}" />
+        <mesh filename="package://wheelbot_description/meshes/arm_segment_a.dae" scale="${1/size_factor} ${1/size_factor} ${1/size_factor}" />
       </geometry>
     </collision>
@@ -86,5 +86,5 @@
       <origin xyz="0 0 ${0.2/size_factor}" rpy="0 ${pi} ${pi}" />
       <geometry>
-        <mesh filename="package://wheeled_robot/meshes/arm_segment_b.dae" scale="${1/size_factor} ${1/size_factor} ${1/size_factor}" />
+        <mesh filename="package://wheelbot_description/meshes/arm_segment_b.dae" scale="${1/size_factor} ${1/size_factor} ${1/size_factor}" />
       </geometry>
       <material name="Orange" />
@@ -92,5 +92,5 @@
     <collision>
       <geometry>
-        <mesh filename="package://wheeled_robot/meshes/arm_segment_b.dae" scale="${1/size_factor} ${1/size_factor} ${1/size_factor}" />
+        <mesh filename="package://wheelbot_description/meshes/arm_segment_b.dae" scale="${1/size_factor} ${1/size_factor} ${1/size_factor}" />
       </geometry>
     </collision>
@@ -107,5 +107,5 @@
       <origin rpy="0 0 ${pi}" />
       <geometry>
-        <mesh filename="package://wheeled_robot/meshes/arm_segment_last.dae" scale="${1/size_factor} ${1/size_factor} ${1/size_factor}" />
+        <mesh filename="package://wheelbot_description/meshes/arm_segment_last.dae" scale="${1/size_factor} ${1/size_factor} ${1/size_factor}" />
       </geometry>
       <material name="Orange"/>
@@ -113,5 +113,5 @@
     <collision>
       <geometry>
-        <mesh filename="package://wheeled_robot/meshes/arm_segment_last.dae" scale="${1/size_factor} ${1/size_factor} ${1/size_factor}" />
+        <mesh filename="package://wheelbot_description/meshes/arm_segment_last.dae" scale="${1/size_factor} ${1/size_factor} ${1/size_factor}" />
       </geometry>
     </collision>
@@ -128,5 +128,5 @@
       <origin rpy="0 0 ${pi}" />
       <geometry>
-        <mesh filename="package://wheeled_robot/meshes/arm_wrist.dae" scale="${1/size_factor} ${1/size_factor} ${1/size_factor}" />
+        <mesh filename="package://wheelbot_description/meshes/arm_wrist.dae" scale="${1/size_factor} ${1/size_factor} ${1/size_factor}" />
       </geometry>
       <material name="Grey"/>
@@ -134,5 +134,5 @@
     <collision>
       <geometry>
-        <mesh filename="package://wheeled_robot/meshes/arm_wrist.dae" scale="${1/size_factor} ${1/size_factor} ${1/size_factor}" />
+        <mesh filename="package://wheelbot_description/meshes/arm_wrist.dae" scale="${1/size_factor} ${1/size_factor} ${1/size_factor}" />
       </geometry>
     </collision>
@@ -149,5 +149,5 @@
       <origin rpy="0 0 ${pi}" />
       <geometry>
-        <mesh filename="package://wheeled_robot/meshes/arm_flanche.dae" scale="${1/size_factor} ${1/size_factor} ${1/size_factor}" />
+        <mesh filename="package://wheelbot_description/meshes/arm_flanche.dae" scale="${1/size_factor} ${1/size_factor} ${1/size_factor}" />
       </geometry>
       <material name="Grey"/>
@@ -155,5 +155,5 @@
     <collision>
       <geometry>
-        <mesh filename="package://wheeled_robot/meshes/arm_flanche.dae" scale="${1/size_factor} ${1/size_factor} ${1/size_factor}" />
+        <mesh filename="package://wheelbot_description/meshes/arm_flanche.dae" scale="${1/size_factor} ${1/size_factor} ${1/size_factor}" />
       </geometry>
     </collision>

File: src/wheeled_robot/wheelbot_description/urdf/materials.xacro (robot description, xacro)
@@ -1,4 +1,4 @@
 <?xml version="1.0"?>
-<robot name="common" xmlns:xacro="http://www.ros.org/wiki/xacro">
+<robot>
   <!-- materials -->
   <material name="Green">
@@ -35,12 +35,3 @@
     <color rgba="0.3058 0.5921 0.7294 1.0"/>
   </material>
-  <!-- macros -->
-  <xacro:macro name="custom_inertia" params="mass ixx:=1 iyy:=1 izz:=1">
-    <inertial>
-      <mass value="${mass}" />
-      <inertia ixx="${ixx}" ixy="0"      ixz="0"
-                            iyy="${iyy}" iyz="0"
-                                         izz="${izz}" />
-    </inertial>
-  </xacro:macro>
 </robot>
