Commit message: Add move 1 meter fwd task

File: src/wheeled_robot/wheelbot_description/urdf/macros.xacro (robot description, xacro)
@@ -22,27 +22,3 @@
           izz="${1/12 * mass * (pow(width, 2) + pow(height, 2))}" />
   </xacro:macro>
-  <xacro:macro name="side_wheel" params="prefix reflect:=1">
-    <link name="${prefix}_wheel">
-      <visual>
-        <material name="Red" />
-        <geometry>
-          <cylinder length="${side_wheel_length}" radius="${side_wheel_radius}" />
-        </geometry>
-      </visual>
-      <collision>
-        <geometry>
-          <cylinder length="${side_wheel_length}" radius="${side_wheel_radius}" />
-        </geometry>
-      </collision>
-      <xacro:cylinder_inertia mass="${side_wheel_mass}"
-        radius="${side_wheel_radius}" length="${side_wheel_length}" />
-    </link>
-    <joint name="base_to_${prefix}_wheel" type="continuous">
-      <parent link="base_link" />
-      <child link="${prefix}_wheel" />
-      <axis xyz="0 0 1" />
-      <origin xyz="${body_width/3} ${reflect * (body_height/2 + side_wheel_length/2)} -${body_depth/2 - side_wheel_offset_z}"
-        rpy="0 ${pi/2} ${pi/2}" />
-    </joint>
-  </xacro:macro>
 </robot>

File: src/wheeled_robot/wheelbot_description/urdf/wheelbot.urdf.xacro (robot description, xacro)
@@ -2,13 +2,13 @@
 <robot name="wheelbot" xmlns:xacro="http://www.ros.org/wiki/xacro">
   <!-- robot parameters -->
-  <xacro:property name="body_mass" value="5" />
+  <xacro:property name="body_mass" value="40" />
   <xacro:property name="body_depth" value="0.2" />
   <xacro:property name="body_width" value="0.5" />
   <xacro:property name="body_height" value="0.3" />
-  <xacro:property name="side_wheel_mass" value="1" />
+  <xacro:property name="side_wheel_mass" value="1.5" />
   <xacro:property name="side_wheel_length" value="0.04" />
   <xacro:property name="side_wheel_radius" value="${3/6 * body_depth}" />
   <xacro:property name="side_wheel_offset_z" value="${1/5 * body_depth}" />
-  <xacro:property name="caster_wheel_mass" value="0.5" />
+  <xacro:property name="caster_wheel_mass" value="1.5" />
   <xacro:property name="caster_wheel_radius" value="${side_wheel_radius / 2}" />
   <xacro:property name="camera_link" value="0.05" />
@@ -17,10 +17,4 @@
   <!-- gazebo -->
   <xacro:include filename="wheelbot.gazebo" />
-  <!-- dummy link workaround (suppress warning message in Gazebo) -->
-  <link name="world" />
-  <joint name="base_to_world" type="fixed">
-    <parent link="world"/>
-    <child link="base_link"/>
-  </joint>
   <!-- base link -->
   <link name="base_link">
@@ -39,6 +33,44 @@
   </link>
   <!-- left and right side wheels -->
-  <xacro:side_wheel prefix="left" reflect="1" />
-  <xacro:side_wheel prefix="right" reflect="-1" />
+  <link name="left_wheel">
+    <visual>
+      <material name="Red" />
+      <geometry>
+        <cylinder length="${side_wheel_length}" radius="${side_wheel_radius}" />
+      </geometry>
+    </visual>
+    <collision>
+      <geometry>
+        <cylinder length="${side_wheel_length}" radius="${side_wheel_radius}" />
+      </geometry>
+    </collision>
+    <xacro:cylinder_inertia mass="${side_wheel_mass}" radius="${side_wheel_radius}" length="${side_wheel_length}" />
+  </link>
+  <joint name="base_to_left_wheel" type="continuous">
+    <parent link="base_link" />
+    <child link="left_wheel" />
+    <axis xyz="0 0 1" />
+    <origin xyz="${body_width/3} ${body_height/2 + side_wheel_length/2} -${body_depth/2 - side_wheel_offset_z}" rpy="0 ${pi/2} ${pi/2}" />
+  </joint>
+  <link name="right_wheel">
+    <visual>
+      <material name="Red" />
+      <geometry>
+        <cylinder length="${side_wheel_length}" radius="${side_wheel_radius}" />
+      </geometry>
+    </visual>
+    <collision>
+      <geometry>
+        <cylinder length="${side_wheel_length}" radius="${side_wheel_radius}" />
+      </geometry>
+    </collision>
+    <xacro:cylinder_inertia mass="${side_wheel_mass}" radius="${side_wheel_radius}" length="${side_wheel_length}" />
+  </link>
+  <joint name="base_to_right_wheel" type="continuous">
+    <parent link="base_link" />
+    <child link="right_wheel" />
+    <axis xyz="0 0 1" />
+    <origin xyz="${body_width/3} -${(body_height/2 + side_wheel_length/2)} -${body_depth/2 - side_wheel_offset_z}" rpy="0 ${pi/2} ${pi/2}" />
+  </joint>
   <!-- 2-DoF caster wheel -->
   <link name="caster_wheel">
@@ -60,8 +92,8 @@
   </link>
   <joint name="base_to_caster_wheel_yaw" type="continuous">
+    <axis xyz="0 0 1" />
     <parent link="base_link" />
     <child link="caster_wheel_virtual" />
     <origin xyz="-${body_width/2} 0 -${body_depth/2 + caster_wheel_radius - side_wheel_offset_z}" />
-    <axis xyz="0 0 1" />
   </joint>
   <link name="caster_wheel_virtual">
@@ -69,7 +101,9 @@
   </link>
   <joint name="base_to_caster_wheel_pitch" type="continuous">
+    <axis xyz="0 1 0" />
     <parent link="caster_wheel_virtual" />
     <child link="caster_wheel" />
-    <axis xyz="0 1 0" />
+    <dynamics damping="0.7" friction="0.1" />
+    <limit effort="100" velocity="50" />
   </joint>
   <!-- camera -->
@@ -140,23 +174,44 @@
     <xacro:custom_inertia mass="1e-5" ixx="1e-6" iyy="1e-6" izz="1e-6" />
   </link>
-  <!-- KUKA LWR manipulator -->
-  <!--
-  <xacro:include filename="$(find wheelbot_description)/urdf/kuka_lwr.xacro" />
-  <joint name="base_to_manipulator" type="fixed">
-    <parent link="base_link" />
-    <child link="arm_base_link" />
-    <origin xyz="0 0 ${body_depth/3}" />
-  </joint>
-  -->
   <!-- Transmissions -->
-  <transmission name="trans_base_to_caster_wheel_yaw">
-    <type>transmission_interface/SimpleTransmission</type>
+  <transmission name="caster_wheel_pitch_trans">
+    <type>transmission_interface/SimpleTransmission</type>
+    <actuator name="caster_wheel_pitch_motor">
+      <hardwareInterface>hardware_interface/EffortJointInterface</hardwareInterface>
+      <mechanicalReduction>1</mechanicalReduction>
+    </actuator>
+    <joint name="base_to_caster_wheel_pitch">
+      <hardwareInterface>hardware_interface/EffortJointInterface</hardwareInterface>
+    </joint>
+  </transmission>
+  <transmission name="caster_wheel_yaw_trans">
+    <type>transmission_interface/SimpleTransmission</type>
+    <actuator name="caster_wheel_yaw_motor">
+      <hardwareInterface>hardware_interface/EffortJointInterface</hardwareInterface>
+      <mechanicalReduction>1</mechanicalReduction>
+    </actuator>
     <joint name="base_to_caster_wheel_yaw">
       <hardwareInterface>hardware_interface/EffortJointInterface</hardwareInterface>
     </joint>
-    <actuator name="base_to_caster_wheel_yaw_motor">
-      <hardwareInterface>hardware_interface/EffortJointInterface</hardwareInterface>
-      <mechanicalReduction>1</mechanicalReduction>
-    </actuator>
+  </transmission>
+  <transmission name="left_wheel_trans">
+    <type>transmission_interface/SimpleTransmission</type>
+    <actuator name="left_wheel_motor">
+      <hardwareInterface>hardware_interface/EffortJointInterface</hardwareInterface>
+      <mechanicalReduction>1</mechanicalReduction>
+    </actuator>
+    <joint name="base_to_left_wheel">
+      <hardwareInterface>hardware_interface/EffortJointInterface</hardwareInterface>
+    </joint>
+  </transmission>
+  <transmission name="right_wheel_trans">
+    <type>transmission_interface/SimpleTransmission</type>
+    <actuator name="right_wheel_motor">
+      <hardwareInterface>hardware_interface/EffortJointInterface</hardwareInterface>
+      <mechanicalReduction>1</mechanicalReduction>
+    </actuator>
+    <joint name="base_to_right_wheel">
+      <hardwareInterface>hardware_interface/EffortJointInterface</hardwareInterface>
+    </joint>
   </transmission>
 </robot>
